File: dds-gen/hardware/DDS-Gen.sch (EAGLE design)
At the start: 36 parts, among them IC1 TL072P, J1 POWER, J2 AVR_SPI_PROG_3X2PTH, J3 I2C CTRL, J4 BNCPTH, Q1 30MHz, U1 ATMEGA328P-PU

Commit message: Updates begin layout of board, switched to ganged resistors
Parts:
- removed R10, R11, R3, R4, R5, R6, R7, R8, R9: 20k, rcl:R-EU_0204/5
- removed R12, R13, R14, R15, R16, R17, R18: 10k, rcl:R-EU_0204/5
- added R23, R24, R25, R26, R27, R28, R29: 10k, rcl:R-EU_0204/5
- added RN1, RN2, RN3, RN4: 10k, resistor-sil:E5R
- R21: device rcl:R-EU_0204/5 -> resistor:R-EU_0204/7
Connections:
- removed net N$13: R17.2, R18.1, R9.1
- removed net N$14: R16.2, R17.1, R8.1
- removed net N$15: R15.2, R16.1, R7.1
- removed net N$16: R14.2, R15.1, R6.1
- removed net N$17: R13.2, R14.1, R5.1
- removed net N$18: R12.2, R13.1, R4.1
- removed net N$19: R11.2, R12.1, R3.1
- removed net N$20: R10.1, R18.2, R19.2
- new net N$25: RN1A.1, RN3A.1
- new net N$26: RN1B.1, RN3B.1
- new net N$27: RN1C.1, RN3C.1
- new net N$28: RN1D.1, RN3D.1
- new net N$29: RN1E.1, RN3E.1
- new net N$30: RN2A.1, RN4A.1
- new net N$31: RN2B.1, RN4B.1
- new net N$32: RN2C.1, RN4C.1
- new net N$33: RN2D.1, RN4D.1
- new net N$34: R23.1, RN4C.2, RN4D.2
- new net N$35: R23.2, R24.1, RN4B.2
- new net N$36: R24.2, R25.1, RN4A.2
- new net N$37: R25.2, R26.1, RN3E.2
- new net N$38: R26.2, R27.1, RN3D.2
- new net N$39: R27.2, R28.1, RN3C.2
- new net N$40: R28.2, R29.1, RN3B.2
- new net N$41: R19.2, R29.2, RN3A.2
- net 0V: now also RN2D.2; no longer R11.1
- net N$10: now also RN2A.2, U1.PD2; no longer R8.2, U1.PD5
- net N$11: now also RN2B.2, U1.PD1; no longer R9.2, U1.PD6
- net N$12: now also RN2C.2, U1.PD0; no longer R10.2, U1.PD7
- net N$5: now also RN1A.2, U1.PD7; no longer R3.2, U1.PD0
- net N$6: now also RN1B.2, U1.PD6; no longer R4.2, U1.PD1
- net N$7: now also RN1C.2, U1.PD5; no longer R5.2, U1.PD2
- net N$8: now also RN1D.2, U1.PD4; no longer R6.2, U1.PD3
- net N$9: now also RN1E.2, U1.PD3; no longer R7.2, U1.PD4
Other:
- moved on the sheet: C5, C6, IC1A, IC1B, J4, R1, R19, R20, R21, R22

Commit message: Layout tweaks and offset control.
Added switchable offset control to output amplifier. Can be switched in or out.
Tweak to layout so pots work in a natual manner (eg clockwise to increase amplitude)
Parts:
- removed C3: 0.1uF, rcl:C-EU025-025X050
- removed R20: 100k, rcl:R-EU_0204/5
- removed R21: 100, resistor:R-EU_0204/7
- removed R23: 10k, rcl:R-EU_0204/5
- added C7: 0.1uF, rcl:C-EU025-025X050
- added R10: 1k, pot:TRIM_EU-S64W
- added R11: 100k, rcl:R-EU_0204/2V
- added R12: 100, rcl:R-EU_0207/12
- added R14: 10k, pot:TRIM_EU-CIP20C-6MM
- added S2: (no value), SparkFun-Switches:SWITCH-SPDT-PTH-11.6X4.0MM
- R1: value 1k -> 10k; device pot:TRIM_EU-S64W -> rcl:R-EU_0204/5
- renumbered R19 to R9, R22 to R13, R24 to R3, R25 to R4, R26 to R5, R27 to R6, R28 to R7, R29 to R8
Connections:
- removed net N$24: R13.A, R21.1
- new net N$13: IC1B.+IN, S2.P
- new net N$15: R14.S, S2.S
- new net N$16: R12.1, R13.E
- net +5V: now also C6.2, R1.2, R10.E, R14.E; no longer C3.2, R1.E, R2.2
- net -5V: now also C7.2, R14.A; no longer C6.2
- net 0V: now also C7.1, R10.A, RN1D.2, S2.O; no longer C3.1, IC1B.+IN, R1.A, RN2D.2
- net N$10: now also RN1A.2; no longer RN2A.2
- net N$11: now also RN1B.2; no longer RN2B.2
- net N$12: now also RN1C.2; no longer RN2C.2
- net N$21: now also R11.1, R12.2; no longer R20.1, R21.2
- net N$23: now also R13.A; no longer R13.E
- net N$29: now also RN2E.1, RN4E.1; no longer RN1E.1, RN3E.1
- net N$3: now also R10.S; no longer R1.S
- net N$34: now also R2.1, RN3C.2, RN3D.2; no longer R23.1, RN4C.2, RN4D.2
- net N$35: now also R2.2, RN3B.2; no longer R23.2, RN4B.2
- net N$36: now also RN3A.2; no longer RN4A.2
- net N$37: now also RN4E.2; no longer RN3E.2
- net N$38: now also RN4D.2; no longer RN3D.2
- net N$39: now also RN4C.2; no longer RN3C.2
- net N$4: now also R11.2; no longer R20.2
- net N$40: now also RN4B.2; no longer RN3B.2
- net N$41: now also RN4A.2; no longer RN3A.2
- net N$5: now also RN2A.2; no longer RN1A.2
- net N$6: now also RN2B.2; no longer RN1B.2
- net N$7: now also RN2C.2; no longer RN1C.2
- net N$8: now also RN2D.2; no longer RN1D.2
- net N$9: now also RN2E.2; no longer RN1E.2
- net RESET: now also R1.1; no longer R2.1
Other:
- note added: "Amplitude (Gain) Control"
- note added: "Offset control (Can be by-passed)"
- note removed: "Amplitude"
- moved on the sheet: C5, C6, R2, RN1A, RN1B, RN1C, RN1D, RN2A, RN2B, RN2C, RN2D, RN3A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

Commit message: Updated Schematic with slit power supply +-9V and 5V
Parts:
- J1: value POWER -> (none); device SparkFun-Connectors:CONN_03POLAR -> SparkFun-Connectors:CONN_06POLAR
Connections:
- removed net +5V: C5.2, C6.2, IC1P.V+, J1.3, J2.2, R1.2, R10.E, R14.E, U1.AREF, U1.AVCC, U1.VCC
- removed net -5V: C7.2, IC1P.V-, J1.1, R14.A
- new net +9V: C6.2, IC1P.V+, J1.4, R10.E, R14.E
- new net -9V: C7.2, IC1P.V-, J1.6, R14.A
- new net VCC: C5.2, J1.1, R1.2, U1.AREF, U1.AVCC, U1.VCC
- net 0V: now also J1.3, J1.5
